File: hardware/breakout-boards/fets/fets.sch (KiCad schematic (older format))
At the start: 37 parts, among them P1 CONN_01X06, P2 CONN_01X06, P3 CONN_01X03, P4 CONN_01X02, Q1 IRF7530, Q2 IRF7530, Q3 IRF7530, Q4 IRF7530, Q5 IRF7530, Q6 IRF7530

Commit message: FET breakoutboard complete, generated gerbers and sent off to fab
Connections:
- net labels added: A_HI_G, A_LO_G, B_HI_G, B_LO_G, C_HI_G, C_LO_G
Changed lines of the file:
@@
 LIBS:contrib
 LIBS:valves
-LIBS:fets-cache
 EELAYER 25 0
 EELAYER END
@@
 Wire Wire Line
 	7700 4950 7700 5000
+Text Label 2450 2850 0    60   ~ 0
+A_LO_G
+Text Label 2450 2000 0    60   ~ 0
+A_HI_G
+Text Label 7400 2000 0    60   ~ 0
+B_HI_G
+Text Label 7400 2850 0    60   ~ 0
+B_LO_G
+Text Label 12150 2000 0    60   ~ 0
+C_HI_G
+Text Label 12150 2850 0    60   ~ 0
+C_LO_G
 $EndSCHEMATC
